File: BaseBoard_Rev0.2/baseboard_0.2.brd (EAGLE design)
At the start: 110 x 97.5 mm, 118 parts, among them Q1 IRLML5203, Q2 IRLML5203, Q3 PDTC114E, Q4 PDTC114E, Q5 PDTC114E, U3 NCP3337MNADJR2G, U4 NCP3337MNADJR2G, X1 CRYSTAL_212M_

Commit message: Added shunt resistor for current measurement
In case of no ammeter
Parts:
- removed JP5: (no value), SparkFun-Passives:1X02
- removed VME_PWR: VEXT_IN, SparkFun-Connectors:BANANA_CONN
- added JP_MEASURE: (no value), jumper:JP2
- added RSH: 10 Ohm 2.5W, rcl:R2512
- added VME_IN: (no value), SparkFun-Connectors:BANANA_CONN
- moved VA_OUT 21.0 mm to (89.4, 71.9)
- moved VA_IN 0.96 mm to (89.3, 86.3)
- moved VMO_GND 0.18 mm to (104.3, 71.9)
Connections:
- new net N$33: JP_MEASURE.1, RSH.1, VA_IN.P$1, VME_IN.P$1
- new net N$35: JP_MEASURE.3, RSH.2
- net VEXT_IN: now also JP_MEASURE.2; no longer JP5.1, JP5.2, VA_IN.P$1, VME_PWR.P$1
Routing:
- net GND: track 645.0 -> 20.8 mm, vias 34 -> 92
- net N$33: track 0.00 -> 39.1 mm
- net VEXT_IN: track 53.3 -> 33.7 mm
- net N$35: track 0.00 -> 5.50 mm
- net V_OPT: track 129.6 -> 131.1 mm
- added copper zone on layer 1, net N$19
- added copper zone on layer 16, net N$19
Other:
- board text added: "1-2 DIRECT"
- board text added: "2-3 SHUNT 10mV/mA"
- board text added: "M+"
- board text added: "M-"
- board text added: "NC AMMETER"
- board text removed: "I+"
- board text removed: "I-"
